File: STM32F405.kicad_sch (KiCad schematic)
At the start: 22 parts, among them SW3 SW_Push, SW4 SW_Push, U3 STM32F405RGTx, Y1 25MHz

Commit message: pcb
Parts:
- removed D6: LED, LED_SMD:LED_0805_2012Metric, symbol Device:LED
- removed R16: 1.2k, Resistor_SMD:R_0603_1608Metric, symbol Device:R
- removed R26: 10k, Resistor_SMD:R_0402_1005Metric, symbol Device:R
- removed SW4: SW_Push, Button_Switch_SMD:SW_Push_SPST_NO_Alps_SKRK, symbol Switch:SW_Push
Connections:
- net CYCLE_LED: now reaches U3.37 (PC6)
- net GND1 renamed GND
- no-connect marks 38 -> 39

Commit message: pcb
Parts:
- SW3: now in the parts list
Changed lines of the file:
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@@
   )
   (symbol (lib_id "Switch:SW_Push") (at 43.18 64.77 90) (unit 1)
-    (in_bom no) (on_board yes) (dnp no)
+    (in_bom yes) (on_board yes) (dnp no)
     (property "Reference" "SW3" (at 31.75 63.5 90)
       (effects (font (size 1.27 1.27)) (justify right))

Commit message: v0.2
Connections:
- net USART2_TX: now reaches U3.16 (PA2)
- net USART2_RX: now reaches U3.17 (PA3)
- no-connect marks 39 -> 37
Changed lines of the file:
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@@
   (no_connect (at 147.32 123.19))
   (no_connect (at 111.76 100.33))
-  (no_connect (at 147.32 64.77))
   (no_connect (at 147.32 120.65))
   (no_connect (at 147.32 115.57))
@@
   (no_connect (at 111.76 90.17))
   (no_connect (at 147.32 97.79))
-  (no_connect (at 147.32 67.31))
   (no_connect (at 147.32 107.95))
   (no_connect (at 147.32 80.01))
@@
     (effects (font (size 1.27 1.27)) (justify left))
   )
+  (hierarchical_label "USART2_TX" (shape output) (at 147.32 64.77 0) (fields_autoplaced)
+    (effects (font (size 1.27 1.27)) (justify left))
+  )
   (hierarchical_label "CYCLE_LED" (shape output) (at 111.76 97.79 180) (fields_autoplaced)
     (effects (font (size 1.27 1.27)) (justify right))
@@
     (effects (font (size 1.27 1.27)) (justify left))
   )
+  (hierarchical_label "USART2_RX" (shape input) (at 147.32 67.31 0) (fields_autoplaced)
+    (effects (font (size 1.27 1.27)) (justify left))
+  )
