File: aif_io.kicad_sch (KiCad schematic)
At the start: 21 parts, among them J1 PWR, J3 CAN, J3 ST-LINK, J4 CAN, J5 AMT21, U1 THVD1420D

Commit message: pcb
Parts:
- added D6: LED, LED_SMD:LED_0805_2012Metric, symbol Device:LED
- added R16: 1.2k, Resistor_SMD:R_0603_1608Metric, symbol Device:R
Connections:
- net GND: now also D6.1 (K)
- new net: D6.2 (A), R16.2
- new net CYCLE_LED: R16.1
Other:
- sheet STM32F405 ports: added CYCLE_LED; removed none
Changed lines of the file:
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@@
     (stroke (width 0) (type default))
   )
+  (wire (pts (xy 142.24 153.67) (xy 142.24 156.21))
+    (stroke (width 0) (type default))
+  )
   (wire (pts (xy 129.54 109.22) (xy 132.08 109.22))
     (stroke (width 0) (type default))
@@
     )
   )
+  (label "CYCLE_LED" (at 142.24 146.05 90) (fields_autoplaced)
+    (effects (font (size 1.27 1.27)) (justify left bottom))
+  )
+  (label "CYCLE_LED" (at 81.28 109.22 0) (fields_autoplaced)
+    (effects (font (size 1.27 1.27)) (justify left bottom))
+  )
   (symbol (lib_id "Connector_Generic:Conn_01x03") (at 115.57 140.97 0) (unit 1)
     (in_bom no) (on_board yes) (dnp no) (fields_autoplaced)
@@
     )
   )
+  (symbol (lib_id "Device:LED") (at 142.24 160.02 270) (mirror x) (unit 1)
+    (in_bom yes) (on_board yes) (dnp no) (fields_autoplaced)
+    (property "Reference" "D6" (at 138.43 160.3375 90)
+      (effects (font (size 1.27 1.27)) (justify right))
+    )
+    (property "Value" "LED" (at 138.43 162.8775 90)
+      (effects (font (size 1.27 1.27)) (justify right))
+    )
+    (property "Footprint" "LED_SMD:LED_0805_2012Metric" (at 142.24 160.02 0)
+      (effects (font (size 1.27 1.27)) hide)
+    )
+    (property "Datasheet" "~" (at 142.24 160.02 0)
+      (effects (font (size 1.27 1.27)) hide)
+    )
+    (property "LCSC" "C34499" (at 142.24 160.02 0)
+      (effects (font (size 1.27 1.27)) hide)
+    )
+    (property "FT Rotation Offset" "" (at 142.24 160.02 0)
+      (effects (font (size 1.27 1.27)) hide)
+    )
+    (pin "1")
+    (pin "2")
+    (instances
+      (project "schematic_MD"
+        (path "/3152684b-d11f-4a9a-8e6c-09965044adbd"
+          (reference "D6") (unit 1)
+        )
+        (path "/3152684b-d11f-4a9a-8e6c-09965044adbd/878f32b7-0d3d-4f49-a9dc-ebc0f2e1c793"
+          (reference "D5") (unit 1)
+        )
+      )
+      (project "aif_io"
+        (path "/9a9f4147-6bcd-4827-a5d0-695037b8e97b/8f28f728-644b-484d-914c-3c6b5b79a75f"
+          (reference "D1") (unit 1)
+        )
+        (path "/9a9f4147-6bcd-4827-a5d0-695037b8e97b"
+          (reference "D1") (unit 1)
+        )
+      )
+    )
+  )
   (symbol (lib_id "Mechanical:MountingHole") (at 120.65 45.72 0) (unit 1)
     (in_bom no) (on_board yes) (dnp no) (fields_autoplaced)
@@
     )
   )
+  (symbol (lib_id "power:GND") (at 142.24 163.83 0) (unit 1)
+    (in_bom yes) (on_board yes) (dnp no) (fields_autoplaced)
+    (property "Reference" "#PWR022" (at 142.24 170.18 0)
+      (effects (font (size 1.27 1.27)) hide)
+    )
+    (property "Value" "GND" (at 142.24 168.91 0)
+      (effects (font (size 1.27 1.27)))
+    )
+    (property "Footprint" "" (at 142.24 163.83 0)
+      (effects (font (size 1.27 1.27)) hide)
+    )
+    (property "Datasheet" "" (at 142.24 163.83 0)
+      (effects (font (size 1.27 1.27)) hide)
+    )
+    (pin "1")
+    (instances
+      (project "aif_io"
+        (path "/9a9f4147-6bcd-4827-a5d0-695037b8e97b/8f28f728-644b-484d-914c-3c6b5b79a75f"
+          (reference "#PWR022") (unit 1)
+        )
+        (path "/9a9f4147-6bcd-4827-a5d0-695037b8e97b"
+          (reference "#PWR021") (unit 1)
+        )
+      )
+    )
+  )
+  (symbol (lib_id "Device:R") (at 142.24 149.86 0) (unit 1)
+    (in_bom yes) (on_board yes) (dnp no)
+    (property "Reference" "R16" (at 139.7 148.59 0)
+      (effects (font (size 1.27 1.27)) (justify right))
+    )
+    (property "Value" "1.2k" (at 139.7 151.13 0)
+      (effects (font (size 1.27 1.27)) (justify right))
+    )
+    (property "Footprint" "Resistor_SMD:R_0603_1608Metric" (at 140.462 149.86 90)
+      (effects (font (size 1.27 1.27)) hide)
+    )
+    (property "Datasheet" "~" (at 142.24 149.86 0)
+      (effects (font (size 1.27 1.27)) hide)
+    )
+    (property "LCSC" "C22765" (at 142.24 149.86 0)
+      (effects (font (size 1.27 1.27)) hide)
+    )
+    (property "FT Rotation Offset" "" (at 142.24 149.86 0)
+      (effects (font (size 1.27 1.27)) hide)
+    )
+    (pin "1")
+    (pin "2")
+    (instances
+      (project "schematic_MD"
+        (path "/3152684b-d11f-4a9a-8e6c-09965044adbd"
+          (reference "R16") (unit 1)
+        )
+        (path "/3152684b-d11f-4a9a-8e6c-09965044adbd/878f32b7-0d3d-4f49-a9dc-ebc0f2e1c793"
+          (reference "R27") (unit 1)
+        )
+      )
+      (project "aif_io"
+        (path "/9a9f4147-6bcd-4827-a5d0-695037b8e97b/8f28f728-644b-484d-914c-3c6b5b79a75f"
+          (reference "R10") (unit 1)
+        )
+        (path "/9a9f4147-6bcd-4827-a5d0-695037b8e97b"
+          (reference "R10") (unit 1)
+        )
+      )
+    )
+  )
   (symbol (lib_id "Device:R") (at 97.79 95.25 0) (unit 1)
     (in_bom yes) (on_board yes) (dnp no)
@@
       (effects (font (size 1.27 1.27)) (justify right))
     )
+    (pin "CYCLE_LED" output (at 81.28 109.22 0)
+      (effects (font (size 1.27 1.27)) (justify right))
+    )

Commit message: v0.2
Parts:
- added C37: 0.1u, Capacitor_SMD:C_0603_1608Metric, symbol Device:C_Small
- added J6: AMT21, Connector_JST:JST_XA_B04B-XASK-1_1x04_P2.50mm_Vertical, symbol Connector_Generic:Conn_01x04
- added JP4: Jumper_2_Open, Connector_PinHeader_2.54mm:PinHeader_1x02_P2.54mm_Vertical, symbol Jumper:Jumper_2_Open
- added R25 (x2): 10, Resistor_SMD:R_0603_1608Metric, symbol Device:R
- added R25: 120, Resistor_SMD:R_0603_1608Metric, symbol Device:R
- added R25 (x2): 10k, Resistor_SMD:R_0603_1608Metric, symbol Device:R
- added U5: THVD1420D, Package_SO:SOIC-8_3.9x4.9mm_P1.27mm, symbol Interface_UART:THVD1420D
Connections:
- net +12V is gone; now on net +5V: J1.2 (Pin_2)
- net +5V: now also C37.1, J6.2 (Pin_2), R25.1, R25.1, U5.8 (VCC)
- net GND: now also C37.2, J6.1 (Pin_1), U5.5 (GND)
- net STM32F405/USART1_RX renamed USART1_RX
- net STM32F405/USART1_TX renamed USART1_TX
- new net: R25.1, U5.7 (B)
- new net: J6.4 (Pin_4), R25.2, R25.2
- new net: J6.3 (Pin_3), JP4.2 (B), R25.2
- new net: JP4.1 (A), R25.1
- new net: R25.1, U5.6 (A)
- new net: R25.2, U5.2 (~{RE}), U5.3 (DE)
- new net USART2_RX: R25.2, U5.1 (RO)
- new net USART2_TX: U5.4 (DI)
Other:
- sheet STM32F405 ports: added USART2_RX, USART2_TX; removed none
- moved on the sheet: C1, H1, H2, H3, H4, J5, JP3, R25, U1
