File: aif_io.kicad_pcb (KiCad board)
At the start: 2 copper layers, 87 parts, among them IC1 ISOW1044BDFMR, IC2 ISOW1044BDFMR, J1 PWR, J2 ST-LINK, J3 CAN, J4 CAN, J5 AMT21, SW1 SW_Push, SW2 SW_Push, U1 THVD1420D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

Commit message: pcb
Parts:
- removed R9: 10k, Resistor_SMD:R_0402_1005Metric
- removed SW2: SW_Push, Button_Switch_SMD:SW_Push_SPST_NO_Alps_SKRK
- added G***: LOGO, logo_pretty:rdclab_small, F.Cu at (79.0, 51.1)
- added REF**: KiCad-Logo2_5mm_SilkScreen, Symbol:KiCad-Logo2_5mm_SilkScreen, F.Cu at (23.8, 54.8)
- moved H1 140.9 mm to (25.0, 25.0)
- moved H2 138.5 mm to (25.0, 45.0)
- moved D2 137.5 mm to (22.8, 31.5)
- moved D3 136.9 mm to (22.8, 35.5)
- moved D4 136.2 mm to (22.8, 39.5)
- moved R11 132.0 mm to (26.2, 31.5), turned to 180 degrees
- moved R12 131.2 mm to (26.2, 35.5), turned to 180 degrees
- moved R13 130.5 mm to (26.2, 39.5), turned to 180 degrees
- moved U4 130.0 mm to (39.0, 27.4), turned to -90 degrees
- moved U3 128.4 mm to (34.4, 33.0)
- moved C15 125.7 mm to (29.5, 28.5), turned to 180 degrees
- moved C18 125.0 mm to (38.0, 23.5), turned to 90 degrees
- moved C17 122.9 mm to (35.5, 28.5), turned to 180 degrees
- moved C16 120.3 mm to (32.2, 37.5)
- moved C36 115.8 mm to (30.0, 44.9), turned to 90 degrees
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Connections:
- C10 pad 2: GND1 -> GND
- C11 pad 2: GND1 -> GND
- C12 pad 2: GND1 -> GND
- C13 pad 2: GND1 -> GND
- C14 pad 2: GND1 -> GND
- C2 pad 2: GND1 -> GND
- C3 pad 2: GND1 -> GND
- C4 pad 2: GND1 -> GND
- C5 pad 2: GND1 -> GND
- C6 pad 2: GND1 -> GND
- C7 pad 2: GND1 -> GND
- C8 pad 2: GND1 -> GND
- C9 pad 2: GND1 -> GND
- D1 pad 1: GND1 -> GND
- R10 pad 1: Net-(U2-PB11) -> /CYCLE_LED
- R8 pad 2: GND1 -> GND
- SW1 pad 1: GND1 -> GND
- U2 pad 12: GND1 -> GND
- U2 pad 18: GND1 -> GND
- U2 pad 21: Net-(U2-PA5) -> unconnected-(U2-PA5-Pad21)
- U2 pad 30: Net-(U2-PB11) -> unconnected-(U2-PB11-Pad30)
- U2 pad 37: unconnected-(U2-PC6-Pad37) -> /CYCLE_LED
- U2 pad 63: GND1 -> GND
- Y1 pad 2: GND1 -> GND
- Y1 pad 4: GND1 -> GND
Routing:
- net +5V: track 0.00 -> 126.6 mm, vias 0 -> 6
- net +3.3V: track 0.00 -> 113.4 mm, vias 0 -> 4
- net GND: track 0.00 -> 43.3 mm, vias 0 -> 185
- net /CAN_Transceiver1/CAN_H: track 0.00 -> 31.6 mm
- net /CAN_Transceiver1/CAN_L: track 0.00 -> 26.4 mm
- net /STM32F405/SWDIO: track 0.00 -> 25.9 mm
- net Net-(U2-NRST): track 0.00 -> 25.7 mm, vias 0 -> 2
- net /CAN_Transceiver2/CAN_TX: track 0.00 -> 21.1 mm
- net Net-(J5-Pin_4): track 0.00 -> 18.7 mm
- net /STM32F405/SWO: track 0.00 -> 18.7 mm
- net /CAN_Transceiver2/CAN_H: track 0.00 -> 18.6 mm
- net /CAN_Transceiver2/CAN_L: track 0.00 -> 16.5 mm
- net /CAN_Transceiver2/CAN_RX: track 0.00 -> 16.0 mm
- net Net-(IC2-VISOIN): track 0.00 -> 15.7 mm
- net /STM32F405/SWCLK: track 0.00 -> 15.7 mm
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- added copper zone on F.Cu, net /CAN_Transceiver1/GND_CAN
- added copper zone on F.Cu, net /CAN_Transceiver2/GND_CAN
- added copper zone on B.Cu, net GND
- added copper zone on F.Cu, net GND
Other:
- board outline added: 60 x 46 mm
- board text added: "12V"
- board text added: "3.3V"
- board text added: "5V"
- board text added: "AIF入出力基板 Ver.0.1 設計：cmos"
- board text added: "AMT21"
- board text added: "CAN1"
- board text added: "CAN2"
- board text added: "ST-LINK"
- board text added: "終端抵抗"
- board text added: "電源表示"

Commit message: pcb
Routing:
- net GND: track 43.3 -> 45.8 mm, vias 185 -> 187
Changed lines of the file:
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@@
     (property "ki_keywords" "connector")
     (attr through_hole exclude_from_pos_files exclude_from_bom)
-    (fp_text reference "J3" (at -3.5 2.8) (layer "F.SilkS")
+    (fp_text reference "J3" (at -3.5 2.7) (layer "F.SilkS")
         (effects (font (size 1 1) (thickness 0.15)))
     )
@@
   (segment (start 65 37) (end 65 35) (width 0.5) (layer "B.Cu") (net 1))
   (segment (start 46.9 50.375075) (end 45.889925 49.365) (width 0.5) (layer "F.Cu") (net 2))
+  (segment (start 54.185 45.485) (end 53 44.3) (width 0.5) (layer "F.Cu") (net 2))
   (segment (start 43.625 51.905) (end 42.7 52.83) (width 0.5) (layer "F.Cu") (net 2))
   (segment (start 48 26.5) (end 48 25) (width 0.25) (layer "F.Cu") (net 2))
   (segment (start 52.7 24.5) (end 53.18 24.5) (width 0.25) (layer "F.Cu") (net 2))
+  (segment (start 58.3 48) (end 57.9 48) (width 0.5) (layer "F.Cu") (net 2))
   (segment (start 47 54) (end 47 53) (width 0.5) (layer "F.Cu") (net 2))
   (segment (start 56.85 47.985) (end 55.009598 47.985) (width 0.5) (layer "F.Cu") (net 2))
@@
   (segment (start 45.889925 49.365) (end 44.65 49.365) (width 0.5) (layer "F.Cu") (net 2))
   (segment (start 40.725 34.5) (end 40.725 35.525) (width 0.5) (layer "F.Cu") (net 2))
-  (segment (start 58.4 46.8) (end 58.4 47.5) (width 0.5) (layer "F.Cu") (net 2))
   (segment (start 56.85 50.525) (end 57.875 50.525) (width 0.5) (layer "F.Cu") (net 2))
   (segment (start 40.725 35.525) (end 40.8 35.6) (width 0.5) (layer "F.Cu") (net 2))
@@
   (segment (start 42.7 52.83) (end 42.7 53.8) (width 0.5) (layer "F.Cu") (net 2))
   (segment (start 40.725 33.475) (end 40.8 33.4) (width 0.5) (layer "F.Cu") (net 2))
-  (segment (start 58.4 47.5) (end 57.915 47.985) (width 0.5) (layer "F.Cu") (net 2))
   (segment (start 46.9 50.8) (end 46.9 51.9) (width 0.5) (layer "F.Cu") (net 2))
   (segment (start 46.9 51.9) (end 46.9 52.9) (width 0.5) (layer "F.Cu") (net 2))
@@
   (segment (start 58.5 49.9) (end 58.5 49.2) (width 0.5) (layer "F.Cu") (net 2))
   (segment (start 58.4 45.97) (end 58.4 46.6) (width 0.5) (layer "F.Cu") (net 2))
+  (segment (start 54.65 45.485) (end 54.185 45.485) (width 0.5) (layer "F.Cu") (net 2))
   (segment (start 56.775 28.925) (end 57.05 28.65) (width 0.25) (layer "F.Cu") (net 2))
   (segment (start 45.4625 40.6) (end 46 40.0625) (width 0.5) (layer "F.Cu") (net 2))
@@
   (segment (start 56.81 45.485) (end 56.85 45.445) (width 0.5) (layer "F.Cu") (net 2))
   (segment (start 53.18 24.5) (end 54.2 23.48) (width 0.25) (layer "F.Cu") (net 2))
+  (segment (start 57.9 48) (end 57.915 47.985) (width 0.5) (layer "F.Cu") (net 2))
   (segment (start 54.925 50.525) (end 54.9 50.5) (width 0.5) (layer "F.Cu") (net 2))
+  (segment (start 58.5 47.8) (end 58.3 48) (width 0.5) (layer "F.Cu") (net 2))
   (segment (start 54.65 45.485) (end 56.81 45.485) (width 0.5) (layer "F.Cu") (net 2))
   (segment (start 44.65 51.905) (end 43.625 51.905) (width 0.5) (layer "F.Cu") (net 2))
-  (segment (start 58.5 46.7) (end 58.4 46.8) (width 0.5) (layer "F.Cu") (net 2))
   (segment (start 45.8 29.6) (end 45.8 29.4) (width 0.25) (layer "F.Cu") (net 2))
+  (segment (start 58.5 46.7) (end 58.4 46.8) (width 0.5) (layer "F.Cu") (net 2))
   (segment (start 57.885 47.985) (end 56.85 47.985) (width 0.5) (layer "F.Cu") (net 2))
   (segment (start 44.075 28.925) (end 45.321827 28.925) (width 0.25) (layer "F.Cu") (net 2))
   (segment (start 42.7 53.8) (end 43.345 54.445) (width 0.5) (layer "F.Cu") (net 2))
+  (segment (start 58.5 46.7) (end 58.5 47.8) (width 0.5) (layer "F.Cu") (net 2))
   (segment (start 45.796827 29.4) (end 45.8 29.6) (width 0.25) (layer "F.Cu") (net 2))
   (segment (start 44.9 40.6) (end 45.4625 40.6) (width 0.5) (layer "F.Cu") (net 2))
@@
   (via (at 69.2 60.1) (size 0.8) (drill 0.4) (layers "F.Cu" "B.Cu") (free) (net 2))
   (via (at 77.6 55.6) (size 0.8) (drill 0.4) (layers "F.Cu" "B.Cu") (free) (net 2))
+  (via (at 53 44.3) (size 0.8) (drill 0.4) (layers "F.Cu" "B.Cu") (net 2))
   (via (at 29.2 29.35) (size 0.8) (drill 0.4) (layers "F.Cu" "B.Cu") (free) (net 2))
   (via (at 27.5 34.1) (size 0.8) (drill 0.4) (layers "F.Cu" "B.Cu") (free) (net 2))
@@
   (via (at 30.7 65.3) (size 0.8) (drill 0.4) (layers "F.Cu" "B.Cu") (free) (net 2))
   (via (at 26.5 65) (size 0.8) (drill 0.4) (layers "F.Cu" "B.Cu") (free) (net 2))
+  (via (at 58.3 48) (size 0.8) (drill 0.4) (layers "F.Cu" "B.Cu") (net 2))
   (via (at 41.4 57.5) (size 0.8) (drill 0.4) (layers "F.Cu" "B.Cu") (free) (net 2))
   (via (at 41.3 36.7) (size 0.8) (drill 0.4) (layers "F.Cu" "B.Cu") (free) (net 2))

Commit message: pcb
Changed lines of the file:
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@@
     (fp_line (start 5 3.2) (end 5 -3.2)
       (stroke (width 0.1) (type solid)) (layer "F.Fab"))
-    (pad "1" thru_hole roundrect (at 0 0) (size 1.7 1.95) (drill 0.95) (layers "*.Cu" "*.Mask") (roundrect_rratio 0.147059)
+    (pad "1" thru_hole roundrect (at 0 0) (size 1.7 1.95) (drill 0.95) (layers "*.Cu" "*.Mask") (roundrect_rratio 0.1470588235)
       (net 2 "GND") (pinfunction "Pin_1") (pintype "passive"))
     (pad "2" thru_hole oval (at 2.5 0) (size 1.7 1.95) (drill 0.95) (layers "*.Cu" "*.Mask")
@@
     (fp_line (start 7.5 3.2) (end 7.5 -3.2)
       (stroke (width 0.1) (type solid)) (layer "F.Fab"))
-    (pad "1" thru_hole roundrect (at 0 0 180) (size 1.7 1.95) (drill 0.95) (layers "*.Cu" "*.Mask") (roundrect_rratio 0.147059)
+    (pad "1" thru_hole roundrect (at 0 0 180) (size 1.7 1.95) (drill 0.95) (layers "*.Cu" "*.Mask") (roundrect_rratio 0.1470588235)
       (net 22 "/CAN_Transceiver2/GND_CAN") (pinfunction "Pin_1") (pintype "passive"))
     (pad "2" thru_hole oval (at 2.5 0 180) (size 1.7 1.95) (drill 0.95) (layers "*.Cu" "*.Mask")
@@
     (fp_line (start 7.5 3.2) (end 7.5 -3.2)
       (stroke (width 0.1) (type solid)) (layer "F.Fab"))
-    (pad "1" thru_hole roundrect (at 0 0 180) (size 1.7 1.95) (drill 0.95) (layers "*.Cu" "*.Mask") (roundrect_rratio 0.147059)
+    (pad "1" thru_hole roundrect (at 0 0 180) (size 1.7 1.95) (drill 0.95) (layers "*.Cu" "*.Mask") (roundrect_rratio 0.1470588235)
       (net 15 "/CAN_Transceiver1/GND_CAN") (pinfunction "Pin_1") (pintype "passive"))
     (pad "2" thru_hole oval (at 2.5 0 180) (size 1.7 1.95) (drill 0.95) (layers "*.Cu" "*.Mask")
@@
     (fp_line (start 10 3.2) (end 10 -3.2)
       (stroke (width 0.1) (type solid)) (layer "F.Fab"))
-    (pad "1" thru_hole roundrect (at 0 0) (size 1.7 1.95) (drill 0.95) (layers "*.Cu" "*.Mask") (roundrect_rratio 0.147059)
+    (pad "1" thru_hole roundrect (at 0 0) (size 1.7 1.95) (drill 0.95) (layers "*.Cu" "*.Mask") (roundrect_rratio 0.1470588235)
       (net 2 "GND") (pinfunction "Pin_1") (pintype "passive"))
     (pad "2" thru_hole oval (at 2.5 0) (size 1.7 1.95) (drill 0.95) (layers "*.Cu" "*.Mask")
@@
     (property "Sheetfile" "STM32F405.kicad_sch")
     (property "Sheetname" "STM32F405")
-    (property "exclude_from_bom" "")
     (property "ki_description" "Push button switch, generic, two pins")
     (property "ki_keywords" "switch normally-open pushbutton push-button")
-    (attr smd exclude_from_bom)
+    (attr smd)
     (fp_text reference "SW1" (at 5.15 0.775) (layer "F.SilkS")
         (effects (font (size 1 1) (thickness 0.15)))
@@
     (fp_line (start 4.11 2.7) (end 3.11 2.7)
       (stroke (width 0.1) (type solid)) (layer "F.Fab"))
-    (pad "1" smd roundrect (at -5.04 -2.28) (size 2.2 1.2) (layers "F.Cu" "F.Paste" "F.Mask") (roundrect_rratio 0.208333)
+    (pad "1" smd roundrect (at -5.04 -2.28) (size 2.2 1.2) (layers "F.Cu" "F.Paste" "F.Mask") (roundrect_rratio 0.2083333333)
       (net 10 "+12V") (pinfunction "IN") (pintype "power_in"))
-    (pad "2" smd roundrect (at -0.415 -1.525) (size 3.05 2.75) (layers "F.Cu" "F.Paste") (roundrect_rratio 0.090909)
+    (pad "2" smd roundrect (at -0.415 -1.525) (size 3.05 2.75) (layers "F.Cu" "F.Paste") (roundrect_rratio 0.09090909091)
       (net 2 "GND") (pinfunction "GND") (pintype "power_in"))
-    (pad "2" smd roundrect (at -0.415 1.525) (size 3.05 2.75) (layers "F.Cu" "F.Paste") (roundrect_rratio 0.090909)
+    (pad "2" smd roundrect (at -0.415 1.525) (size 3.05 2.75) (layers "F.Cu" "F.Paste") (roundrect_rratio 0.09090909091)
       (net 2 "GND") (pinfunction "GND") (pintype "power_in"))
-    (pad "2" smd roundrect (at 1.26 0) (size 6.4 5.8) (layers "F.Cu" "F.Mask") (roundrect_rratio 0.043103)
+    (pad "2" smd roundrect (at 1.26 0) (size 6.4 5.8) (layers "F.Cu" "F.Mask") (roundrect_rratio 0.04310293103)
       (net 2 "GND") (pinfunction "GND") (pintype "power_in"))
-    (pad "2" smd roundrect (at 2.935 -1.525) (size 3.05 2.75) (layers "F.Cu" "F.Paste") (roundrect_rratio 0.090909)
+    (pad "2" smd roundrect (at 2.935 -1.525) (size 3.05 2.75) (layers "F.Cu" "F.Paste") (roundrect_rratio 0.09090909091)
       (net 2 "GND") (pinfunction "GND") (pintype "power_in"))
-    (pad "2" smd roundrect (at 2.935 1.525) (size 3.05 2.75) (layers "F.Cu" "F.Paste") (roundrect_rratio 0.090909)
+    (pad "2" smd roundrect (at 2.935 1.525) (size 3.05 2.75) (layers "F.Cu" "F.Paste") (roundrect_rratio 0.09090909091)
       (net 2 "GND") (pinfunction "GND") (pintype "power_in"))
-    (pad "3" smd roundrect (at -5.04 2.28) (size 2.2 1.2) (layers "F.Cu" "F.Paste" "F.Mask") (roundrect_rratio 0.208333)
+    (pad "3" smd roundrect (at -5.04 2.28) (size 2.2 1.2) (layers "F.Cu" "F.Paste" "F.Mask") (roundrect_rratio 0.2083333333)
       (net 1 "+5V") (pinfunction "OUT") (pintype "power_out"))
     (model "${KICAD6_3DMODEL_DIR}/Package_TO_SOT_SMD.3dshapes/TO-252-2.wrl"
@@
     (fp_line (start 1 0.625) (end -1 0.625)
       (stroke (width 0.1) (type solid)) (layer "F.Fab"))
-    (pad "1" smd roundrect (at -0.9125 0) (size 1.025 1.4) (layers "F.Cu" "F.Paste" "F.Mask") (roundrect_rratio 0.243902)
+    (pad "1" smd roundrect (at -0.9125 0) (size 1.025 1.4) (layers "F.Cu" "F.Paste" "F.Mask") (roundrect_rratio 0.243902439)
       (net 8 "+3.3V") (pinfunction "1") (pintype "passive"))
-    (pad "2" smd roundrect (at 0.9125 0) (size 1.025 1.4) (layers "F.Cu" "F.Paste" "F.Mask") (roundrect_rratio 0.243902)
+    (pad "2" smd roundrect (at 0.9125 0) (size 1.025 1.4) (layers "F.Cu" "F.Paste" "F.Mask") (roundrect_rratio 0.243902439)
       (net 9 "VDDA") (pinfunction "2") (pintype "passive"))
     (model "${KICAD6_3DMODEL_DIR}/Resistor_SMD.3dshapes/R_0805_2012Metric.wrl"
@@
   (segment (start 31.5 37.5) (end 31.45 37.5) (width 0.5) (layer "F.Cu") (net 1))
   (segment (start 29.375 35.425) (end 31.45 37.5) (width 0.5) (layer "F.Cu") (net 1))
+  (segment (start 32.610046 29.5) (end 35.275 29.5) (width 0.5) (layer "F.Cu") (net 1))
   (segment (start 41.5 54.5) (end 41.5 45.5) (width 0.5) (layer "F.Cu") (net 1))
   (segment (start 43.465 56.465) (end 41.5 54.5) (width 0.5) (layer "F.Cu") (net 1))
-  (segment (start 32.610046 29.5) (end 35.275 29.5) (width 0.5) (layer "F.Cu") (net 1))
   (segment (start 53.15 52.985) (end 53.15 50.65) (width 0.5) (layer "F.Cu") (net 1))
   (segment (start 49.015 53.515) (end 49.5 54) (width 0.25) (layer "F.Cu") (net 1))
@@
   (segment (start 49.5 51) (end 49.5 54) (width 0.5) (layer "F.Cu") (net 1))
   (segment (start 64 42.5) (end 65 41.5) (width 0.5) (layer "F.Cu") (net 1))
+  (segment (start 31.45 37.5) (end 31.6 37.35) (width 0.5) (layer "F.Cu") (net 1))
   (segment (start 29 37.5) (end 31.45 37.5) (width 0.25) (layer "F.Cu") (net 1))
   (segment (start 59.825 41) (end 59.825 41.175) (width 0.25) (layer "F.Cu") (net 1))
@@
   (segment (start 49.5 54) (end 49.5 55) (width 0.5) (layer "F.Cu") (net 1))
   (segment (start 62.975 35.3) (end 58.8 35.3) (width 0.25) (layer "F.Cu") (net 1))
-  (segment (start 35.275 29.5) (end 36.275 28.5) (width 0.5) (layer "F.Cu") (net 1))
   (segment (start 58.095 34.595) (end 58.095 34) (width 0.25) (layer "F.Cu") (net 1))
   (segment (start 27 35.5) (end 29 37.5) (width 0.25) (layer "F.Cu") (net 1))
@@
   (segment (start 48.95 47.875) (end 48.325 48.5) (width 0.25) (layer "F.Cu") (net 1))
   (segment (start 51.65 50.85) (end 52.5 50) (width 0.25) (layer "F.Cu") (net 1))
-  (segment (start 31.45 37.5) (end 31.45 30.660046) (width 0.5) (layer "F.Cu") (net 1))
+  (segment (start 31.6 37.35) (end 31.6 30.510046) (width 0.5) (layer "F.Cu") (net 1))
+  (segment (start 31.6 30.510046) (end 32.610046 29.5) (width 0.5) (layer "F.Cu") (net 1))
   (segment (start 55.5 42.5) (end 56 43) (width 0.25) (layer "F.Cu") (net 1))
   (segment (start 63.5 34.775) (end 62.975 35.3) (width 0.25) (layer "F.Cu") (net 1))
-  (segment (start 31.45 30.660046) (end 32.610046 29.5) (width 0.5) (layer "F.Cu") (net 1))
+  (segment (start 35.275 29.5) (end 36.275 28.5) (width 0.5) (layer "F.Cu") (net 1))
   (segment (start 63.5 34.775) (end 64.775 34.775) (width 0.25) (layer "F.Cu") (net 1))
   (segment (start 54.485 42.5) (end 55.5 42.5) (width 0.25) (layer "F.Cu") (net 1))

Commit message: v0.2
Parts:
- removed C16: 0.1u, Capacitor_SMD:C_0603_1608Metric
- removed D2: LED, LED_SMD:LED_0603_1608Metric
- removed R11: 10k, Resistor_SMD:R_0603_1608Metric
- removed REF**: KiCad-Logo2_5mm_SilkScreen, Symbol:KiCad-Logo2_5mm_SilkScreen
- removed U3: L7805, Package_TO_SOT_SMD:TO-252-2
- added C37: 0.1u, Capacitor_SMD:C_0603_1608Metric, F.Cu at (55.5, 20.5)
- added J6: AMT21, Connector_JST:JST_XA_B04B-XASK-1_1x04_P2.50mm_Vertical, F.Cu at (61.0, 21.5)
- added JP4: Jumper_2_Open, Connector_PinHeader_2.54mm:PinHeader_1x02_P2.54mm_Vertical, F.Cu at (75.6, 20.0)
- added R16: 10k, Resistor_SMD:R_0603_1608Metric, F.Cu at (44.7, 23.8)
- added R17: 10, Resistor_SMD:R_0603_1608Metric, F.Cu at (55.4, 23.2)
- added R18: 10, Resistor_SMD:R_0603_1608Metric, F.Cu at (55.4, 24.8)
- added R19: 120, Resistor_SMD:R_0603_1608Metric, F.Cu at (72.2, 22.2)
- added R9: 10k, Resistor_SMD:R_0603_1608Metric, F.Cu at (44.8, 21.0)
- added U5: THVD1420D, Package_SO:SOIC-8_3.9x4.9mm_P1.27mm, F.Cu at (50.0, 23.0)
- C15: value 0.47u -> 100u; footprint Capacitor_SMD:C_0603_1608Metric -> Capacitor_THT:C_Radial_D6.3mm_H11.0mm_P2.50mm
- moved G*** 60.3 mm to (27.9, 19.0), turned to 0 degrees
- moved C15 8.96 mm to (34.0, 36.2)
- moved C17 7.29 mm to (38.2, 35.2)
- moved D3 6.50 mm to (22.8, 42.0)
- moved R12 6.50 mm to (26.2, 42.0)
- moved C1 5.00 mm to (63.5, 39.0)
- moved C10 5.00 mm to (42.0, 34.5)
- moved C11 5.00 mm to (47.5, 29.0)
- moved C12 5.00 mm to (42.0, 41.0)
- moved C13 5.00 mm to (55.0, 43.0)
- moved C14 5.00 mm to (56.0, 32.5)
- moved C18 5.00 mm to (38.0, 28.5)
- moved C19 5.00 mm to (51.6, 60.2)
- moved C2 5.00 mm to (42.5, 44.0)
- moved C20 5.00 mm to (53.1, 60.2)
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Connections:
- net /STM32F405/USART1_RX renamed /USART1_RX
- net /STM32F405/USART1_TX renamed /USART1_TX
- C15 pad 1: +12V -> +5V
- J1 pad 2: +12V -> +5V
- U2 pad 16: unconnected-(U2-PA2-Pad16) -> /USART2_TX
- U2 pad 17: unconnected-(U2-PA3-Pad17) -> /USART2_RX
Routing:
- net +5V: track 126.6 -> 184.7 mm
- net Net-(J6-Pin_3): track 0.00 -> 31.6 mm
- net Net-(J6-Pin_4): track 0.00 -> 20.5 mm
- net /USART2_RX: track 0.00 -> 16.7 mm
- net +12V: track 15.0 -> 0.00 mm
- net /USART2_TX: track 0.00 -> 9.76 mm
- net Net-(JP4-A): track 0.00 -> 3.93 mm
- net +3.3V: track 113.4 -> 109.5 mm, vias 4 -> 8
- net Net-(U5-DE): track 0.00 -> 3.34 mm
- net Net-(U5-A): track 0.00 -> 2.60 mm
- net Net-(U5-B): track 0.00 -> 2.47 mm
- net /USART1_RX: track 12.1 -> 14.1 mm
- net Net-(D2-A): track 1.78 -> 0.00 mm
- net GND: vias 187 -> 240
Other:
- board size 60 x 46 mm -> 60 x 54 mm
- board text added: "AIF入出力基板 Ver.0.2 設計：cmos"
- board text removed: "12V"
- board text removed: "AIF入出力基板 Ver.0.1 設計：cmos"

Commit message: pcb
Routing:
- net GND: vias 240 -> 244
Changed lines of the file:
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@@
   (via (at 72.2 62.7) (size 0.8) (drill 0.4) (layers "F.Cu" "B.Cu") (free) (net 2))
   (via (at 21.2 47.5) (size 0.8) (drill 0.4) (layers "F.Cu" "B.Cu") (free) (net 2))
+  (via (at 75.9 25.5) (size 0.8) (drill 0.4) (layers "F.Cu" "B.Cu") (free) (net 2))
   (via (at 61.7 36.7) (size 0.8) (drill 0.4) (layers "F.Cu" "B.Cu") (free) (net 2))
   (via (at 51.25 25.25) (size 0.8) (drill 0.4) (layers "F.Cu" "B.Cu") (free) (net 2))
@@
   (via (at 58.5 54.2) (size 0.8) (drill 0.4) (layers "F.Cu" "B.Cu") (net 2))
   (via (at 22.7 21.4) (size 0.8) (drill 0.4) (layers "F.Cu" "B.Cu") (free) (net 2))
+  (via (at 69 47.8) (size 0.8) (drill 0.4) (layers "F.Cu" "B.Cu") (free) (net 2))
   (via (at 34.7 23.9) (size 0.8) (drill 0.4) (layers "F.Cu" "B.Cu") (free) (net 2))
   (via (at 21.9 57.1) (size 0.8) (drill 0.4) (layers "F.Cu" "B.Cu") (free) (net 2))
@@
   (via (at 33.9 61.9) (size 0.8) (drill 0.4) (layers "F.Cu" "B.Cu") (free) (net 2))
   (via (at 46.9 55.8) (size 0.8) (drill 0.4) (layers "F.Cu" "B.Cu") (net 2))
-  (via (at 69.9 49.8) (size 0.8) (drill 0.4) (layers "F.Cu" "B.Cu") (free) (net 2))
+  (via (at 69.5 50.4) (size 0.8) (drill 0.4) (layers "F.Cu" "B.Cu") (free) (net 2))
   (via (at 57.05 33.65) (size 0.8) (drill 0.4) (layers "F.Cu" "B.Cu") (net 2))
   (via (at 62.7 70.2) (size 0.8) (drill 0.4) (layers "F.Cu" "B.Cu") (free) (net 2))
+  (via (at 40.2 42.4) (size 0.8) (drill 0.4) (layers "F.Cu" "B.Cu") (free) (net 2))
   (via (at 66.7 48.1) (size 0.8) (drill 0.4) (layers "F.Cu" "B.Cu") (free) (net 2))
   (via (at 23.9 32.8) (size 0.8) (drill 0.4) (layers "F.Cu" "B.Cu") (free) (net 2))
@@
   (via (at 63.4 37.2) (size 0.8) (drill 0.4) (layers "F.Cu" "B.Cu") (free) (net 2))
   (via (at 49.35 40.6) (size 0.8) (drill 0.4) (layers "F.Cu" "B.Cu") (free) (net 2))
+  (via (at 74.3 23.5) (size 0.8) (drill 0.4) (layers "F.Cu" "B.Cu") (free) (net 2))
   (via (at 21.8 62.7) (size 0.8) (drill 0.4) (layers "F.Cu" "B.Cu") (free) (net 2))
   (via (at 40.3 51) (size 0.8) (drill 0.4) (layers "F.Cu" "B.Cu") (free) (net 2))
@@
   (via (at 54.9 28.9) (size 0.8) (drill 0.4) (layers "F.Cu" "B.Cu") (free) (net 2))
   (via (at 61.4 26.4) (size 0.8) (drill 0.4) (layers "F.Cu" "B.Cu") (free) (net 2))
-  (via (at 32.8 68.5) (size 0.8) (drill 0.4) (layers "F.Cu" "B.Cu") (free) (net 2))
+  (via (at 33 67.5) (size 0.8) (drill 0.4) (layers "F.Cu" "B.Cu") (free) (net 2))
   (via (at 48.8 65) (size 0.8) (drill 0.4) (layers "F.Cu" "B.Cu") (free) (net 2))
   (via (at 45.8 34.6) (size 0.8) (drill 0.4) (layers "F.Cu" "B.Cu") (net 2))
